File: BrakeOnly/BrakeOnly.kicad_pcb (KiCad board)
At the start: 2 copper layers, 88.4 x 25.4 mm, 0 parts

Commit message: Completed light boards.
Parts:
- added D101: LED, LED_SMD:LED_Cree-XB, F.Cu at (104.0, 69.8)
- added D102: LED, LED_SMD:LED_Cree-XB, F.Cu at (119.4, 69.8)
- added D103: LED, LED_SMD:LED_Cree-XB, F.Cu at (134.6, 69.8)
- added D104: LED, LED_SMD:LED_Cree-XB, F.Cu at (147.3, 69.8)
- added D105: LED, LED_SMD:LED_Cree-XB, F.Cu at (158.8, 69.8)
- added J0: C-, SpadeLugs:197054303, B.Cu at (95.2, 72.4)
- added J101: Brake+, SpadeLugs:197054303, B.Cu at (166.4, 72.1)
- added R101: 6.2, Resistor_SMD:R_2010_5025Metric, F.Cu at (162.1, 72.4)
Routing:
- added copper zone on F.Cu, net GNDPWR
- added copper zone on F.Cu, net Net-(D101-Pad2)
- added copper zone on F.Cu, net Net-(D102-Pad2)
- added copper zone on F.Cu, net Net-(D103-Pad2)
- added copper zone on F.Cu, net Net-(D104-Pad2)
- added copper zone on F.Cu, net Net-(D105-Pad2)
- added copper zone on F.Cu, net Net-(J101-Pad1)
