File: BrakeOnly/BrakeOnly.kicad_sch (KiCad schematic)
At the start: 1 part, among them J0 C-

Commit message: Completed light boards.
Parts:
- added D101, D102, D103, D104, D105: LED, LED_SMD:LED_Cree-XB, symbol Device:LED
- added J101: Brake+, SpadeLugs:197054303, symbol SpadeLugs:19705-4303
- added R101: 6.2, Resistor_SMD:R_2010_5025Metric, symbol Device:R
Connections:
- net GNDPWR: now also D101.1 (K)
- new net: D101.2 (A), D102.1 (K)
- new net: D102.2 (A), D103.1 (K)
- new net: D104.2 (A), D105.1 (K)
- new net: D105.2 (A), R101.1
- new net: J101.1, J101.2, R101.2
- new net: D103.2 (A), D104.1 (K)
Other:
- moved on the sheet: J0
