File: MarkerTurnSignal/MarkerTurnSignal.kicad_pcb (KiCad board)
At the start: 2 copper layers, 88.4 x 25.4 mm, 0 parts

Commit message: Completed light boards.
Parts:
- added D101: LED, LED_SMD:LED_Avago_PLCC4_3.2x2.8mm_CW, F.Cu at (140.2, 69.4)
- added D102: LED, LED_SMD:LED_Avago_PLCC4_3.2x2.8mm_CW, F.Cu at (122.4, 69.9)
- added D103: LED, LED_SMD:LED_Avago_PLCC4_3.2x2.8mm_CW, F.Cu at (147.9, 69.4)
- added D104: LED, LED_SMD:LED_Avago_PLCC4_3.2x2.8mm_CW, F.Cu at (114.8, 69.9)
- added D105: LED, LED_SMD:LED_Avago_PLCC4_3.2x2.8mm_CW, F.Cu at (155.5, 69.4)
- added D106: LED, LED_SMD:LED_Avago_PLCC4_3.2x2.8mm_CW, F.Cu at (107.2, 69.9)
- added D107: LED, LED_SMD:LED_Avago_PLCC4_3.2x2.8mm_CW, F.Cu at (162.6, 69.4)
- added D108: LED, LED_SMD:LED_Avago_PLCC4_3.2x2.8mm_CW, F.Cu at (100.1, 69.9)
- added J0: C-, SpadeLugs:197054303, B.Cu at (132.1, 66.5)
- added J101: Turn+, SpadeLugs:197054303, B.Cu at (169.2, 66.5)
- added J102: Marker+, SpadeLugs:197054303, B.Cu at (93.5, 66.5)
- added R101: 47, Resistor_SMD:R_0603_1608Metric, F.Cu at (163.8, 64.5)
- added R102: 47, Resistor_SMD:R_0603_1608Metric, F.Cu at (97.9, 75.2)
Routing:
- net GNDPWR: track 0.00 -> 30.0 mm
- net Net-(J101-Pad1): track 0.00 -> 10.5 mm
- net Net-(J102-Pad1): track 0.00 -> 10.1 mm
- net Net-(D104-Pad2): track 0.00 -> 9.14 mm
- net Net-(D103-Pad2): track 0.00 -> 9.12 mm
- net Net-(D101-Pad2): track 0.00 -> 9.12 mm
- net Net-(D102-Pad2): track 0.00 -> 9.10 mm
- net Net-(D106-Pad2): track 0.00 -> 8.61 mm
- net Net-(D105-Pad2): track 0.00 -> 8.61 mm
- net Net-(D108-Pad2): track 0.00 -> 4.62 mm
- net Net-(D107-Pad2): track 0.00 -> 4.56 mm
- added copper zone on B.Cu, net GNDPWR
