File: TaillightBoard/TaillightBoard.kicad_pcb (KiCad board)
At the start: 2 copper layers, 88.4 x 25.4 mm, 0 parts

Commit message: Completed light boards.
Parts:
- added D101: LED, LED_SMD:LED_Cree-PLCC4_3.2x2.8mm_CCW, F.Cu at (93.2, 75.5)
- added D102: LED, LED_SMD:LED_Cree-PLCC4_3.2x2.8mm_CCW, F.Cu at (164.9, 70.4)
- added D103: LED, LED_SMD:LED_Avago_PLCC4_3.2x2.8mm_CW, F.Cu at (93.0, 68.8)
- added D104: LED, LED_SMD:LED_Cree-PLCC4_3.2x2.8mm_CCW, F.Cu at (98.8, 75.5)
- added D105: LED, LED_SMD:LED_Avago_PLCC4_3.2x2.8mm_CW, F.Cu at (98.6, 68.8)
- added D106: LED, LED_SMD:LED_Cree-PLCC4_3.2x2.8mm_CCW, F.Cu at (157.5, 70.6)
- added D107: LED, LED_SMD:LED_Avago_PLCC4_3.2x2.8mm_CW, F.Cu at (104.2, 68.8)
- added D108: LED, LED_SMD:LED_Cree-PLCC4_3.2x2.8mm_CCW, F.Cu at (104.1, 75.7)
- added D109: LED, LED_SMD:LED_Cree-PLCC4_3.2x2.8mm_CCW, F.Cu at (151.4, 70.6)
- added D110: LED, LED_SMD:LED_Avago_PLCC4_3.2x2.8mm_CW, F.Cu at (110.3, 68.8)
- added D111: LED, LED_SMD:LED_Cree-PLCC4_3.2x2.8mm_CCW, F.Cu at (109.7, 75.7)
- added D112: LED, LED_SMD:LED_Cree-PLCC4_3.2x2.8mm_CCW, F.Cu at (145.3, 70.6)
- added J0: C-, SpadeLugs:197054303, B.Cu at (93.5, 63.0)
- added J101: Turn+, SpadeLugs:197054303, B.Cu at (126.0, 69.1)
- added J102: Brake+, SpadeLugs:197054303, B.Cu at (126.5, 75.2)
- added J103: Tail+, SpadeLugs:197054303, B.Cu at (134.6, 64.0)
- added R101: 47, Resistor_SMD:R_0603_1608Metric, F.Cu at (115.5, 68.1)
- added R102: 47, Resistor_SMD:R_0603_1608Metric, F.Cu at (115.1, 76.7)
- added R103: 47, Resistor_SMD:R_0603_1608Metric, F.Cu at (139.7, 69.6)
Routing:
- net GNDPWR: track 0.00 -> 22.0 mm, vias 0 -> 1
- net Net-(J102-Pad1): track 0.00 -> 11.2 mm
- net Net-(J101-Pad1): track 0.00 -> 10.1 mm
- net Net-(J103-Pad1): track 0.00 -> 9.55 mm
- net Net-(D102-Pad1): track 0.00 -> 8.87 mm
- net Net-(D107-Pad2): track 0.00 -> 7.60 mm
- net Net-(D112-Pad1): track 0.00 -> 7.54 mm
- net Net-(D106-Pad1): track 0.00 -> 7.50 mm
- net Net-(D109-Pad1): track 0.00 -> 7.50 mm
- net Net-(D111-Pad1): track 0.00 -> 7.35 mm
- net Net-(D103-Pad2): track 0.00 -> 7.10 mm
- net Net-(D105-Pad2): track 0.00 -> 7.09 mm
- net Net-(D101-Pad1): track 0.00 -> 6.99 mm
- net Net-(D108-Pad1): track 0.00 -> 6.99 mm
- net Net-(D104-Pad1): track 0.00 -> 6.79 mm
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- added copper zone on B.Cu, net GNDPWR
