File: TaillightBoard/TaillightBoard.kicad_sch (KiCad schematic)
At the start: 1 part, among them J0 C-

Commit message: Completed light boards.
Parts:
- added D101, D102, D104, D106, D108, D109, D111, D112: LED, LED_SMD:LED_Cree-PLCC4_3.2x2.8mm_CCW, symbol Device:LED
- added D103, D105, D107, D110: LED, LED_SMD:LED_Avago_PLCC4_3.2x2.8mm_CW, symbol Device:LED
- added J101: Turn+, SpadeLugs:197054303, symbol SpadeLugs:19705-4303
- added J102: Brake+, SpadeLugs:197054303, symbol SpadeLugs:19705-4303
- added J103: Tail+, SpadeLugs:197054303, symbol SpadeLugs:19705-4303
- added R101, R102, R103: 47, Resistor_SMD:R_0603_1608Metric, symbol Device:R
Connections:
- net GNDPWR: now also D101.4 (K), D102.4 (K), D103.1 (K), D103.3 (K), D103.4 (K)
- new net: D107.2 (A), D110.1 (K), D110.3 (K), D110.4 (K)
- new net: D110.2 (A), R101.1
- new net: D112.1 (A), D112.2 (A), D112.3 (A), R103.1
- new net: D109.1 (A), D109.2 (A), D109.3 (A), D112.4 (K)
- new net: D102.1 (A), D102.2 (A), D102.3 (A), D106.4 (K)
- new net: J101.1, J101.2, R101.2
- new net: D104.1 (A), D104.2 (A), D104.3 (A), D108.4 (K)
- new net: D101.1 (A), D101.2 (A), D101.3 (A), D104.4 (K)
- new net: D105.2 (A), D107.1 (K), D107.3 (K), D107.4 (K)
- new net: D103.2 (A), D105.1 (K), D105.3 (K), D105.4 (K)
- new net: D108.1 (A), D108.2 (A), D108.3 (A), D111.4 (K)
- new net: J103.1, J103.2, R103.2
- new net: D106.1 (A), D106.2 (A), D106.3 (A), D109.4 (K)
- new net: D111.1 (A), D111.2 (A), D111.3 (A), R102.1
- new net: J102.1, J102.2, R102.2
